File: arduino_midi2cv_gate_unbuffered.sch (EAGLE design)
At the start: 10 parts, among them IC1 MCP4921 pin numbers incorrect

Commit message: power decoupling and output shorting protection
Parts:
- added C1, C2: 100n, capacitor-wima:C2,5-3
- added C3: 10u, adafruit:CPOL-US085CS-1AR
- added R3, R4: 100, rcl:R-EU_0204/2V
Connections:
- removed net N$8: CV_OUT.3, IC1.VOUT
- new net N$1: IC1.VOUT, R3.1
- new net N$10: GATE_OUT.3, R4.2
- new net N$4: CV_OUT.3, R3.2
- net D2: now also R4.1; no longer GATE_OUT.3
- net GND: now also C1.2, C2.1, C3.-
- net N$5: now also C1.1
- net VCC: now also C2.2, C3.+
Other:
- note added: "Arduino Pro Micro MIDI to CV/gate 5V USB powered"
- note removed: "Arduino Pro Micro"
- moved on the sheet: CV_OUT, GATE_OUT
